File: RTI-RoR-Hardware/RTI-RoR.sch (EAGLE design)
At the start: 30 parts, among them IC2 74LVC244

Commit message: Adding the at park pins to both PCB for the Arduino DUE.
Parts:
- added X7: (no value), con-ptr500:AK500/2
Connections:
- new net AT_PARK_PIN: PCB1.A5, X7-1.KL
- new net AT_PARK_PIN_LOOP: PCB1.A4, X7-2.KL
- new net XBEE_RESET: PCB1.8
Changed lines of the file:
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@@
 <part name="R2" library="rti" deviceset="R-EU" device="'0805'" value="100K 0.1%"/>
 <part name="C3" library="rti" deviceset="C-EU" device="'0805'" value="10uF"/>
+<part name="X7" library="con-ptr500" deviceset="AK500/2" device=""/>
 </parts>
 <sheets>
@@
 <instance part="R2" gate="G$1" x="5.08" y="129.54" rot="R90"/>
 <instance part="C3" gate="G$1" x="185.42" y="53.34"/>
+<instance part="X7" gate="-1" x="43.18" y="22.86" rot="R180"/>
+<instance part="X7" gate="-2" x="43.18" y="27.94" rot="R180"/>
 </instances>
 <busses>
@@
 </segment>
 </net>
+<net name="XBEE_RESET" class="0">
+<segment>
+<wire x1="137.16" y1="66.04" x2="134.62" y2="66.04" width="0.1524" layer="91"/>
+<label x="137.16" y="66.04" size="1.016" layer="95" xref="yes"/>
+<pinref part="PCB1" gate="G$1" pin="8"/>
+</segment>
+</net>
 <net name="N$5" class="0">
 <segment>
@@
 </segment>
 </net>
+<net name="AT_PARK_PIN_LOOP" class="0">
+<segment>
+<pinref part="PCB1" gate="G$1" pin="A4"/>
+<wire x1="73.66" y1="43.18" x2="76.2" y2="43.18" width="0.1524" layer="91"/>
+<label x="73.66" y="43.18" size="1.016" layer="95" rot="R180" xref="yes"/>
+</segment>
+<segment>
+<pinref part="X7" gate="-2" pin="KL"/>
+<wire x1="35.56" y1="27.94" x2="38.1" y2="27.94" width="0.1524" layer="91"/>
+<label x="35.56" y="27.94" size="1.016" layer="95" rot="R180" xref="yes"/>
+</segment>
+</net>
+<net name="AT_PARK_PIN" class="0">
+<segment>
+<pinref part="PCB1" gate="G$1" pin="A5"/>
+<wire x1="73.66" y1="40.64" x2="76.2" y2="40.64" width="0.1524" layer="91"/>
+<label x="73.66" y="40.64" size="1.016" layer="95" rot="R180" xref="yes"/>
+</segment>
+<segment>
+<pinref part="X7" gate="-1" pin="KL"/>
+<wire x1="35.56" y1="22.86" x2="38.1" y2="22.86" width="0.1524" layer="91"/>
+<label x="35.56" y="22.86" size="1.016" layer="95" rot="R180" xref="yes"/>
+</segment>
+</net>
