File: Hardware/RTI-RoR.sch (EAGLE design)
At the start: 31 parts, among them IC2 74LVC244

Commit message: Use the same board as the dome.
Parts:
- removed IC2: 74LVC244, rti:74LVC244
- removed JP4: (no value), jumper:JP1E
- removed U$2: STL-140-2, rti:STL-140-2
- removed U$3: STL-140-6, rti:STL-140-6
- added C5, C6, C7, C8, C9: 100nF, rti:C-EU'0805'
- added IC1: 24AA128ST, microchip:24AA128ST
- added IC3: FT232RL, ftdichip:FT232RL
- added IC5: 74LVC245, rti:74LVC245
- added IC6: 74ABT245, rti:74LVC245
- added R1, R3: 1K, rti:R-EU'0805'
- added R11: 10K, rti:R-EU'0805'
- added R12, R20, R21, R22, R9: 4.7K, rti:R-EU'0805'
- added X11, X12, X8: (no value), con-ptr500:AK500/2
- added X13: PN61729-S, con-berg:PN61729-S
- added XB1: XBEE, maxstream:XBEE
- R13, R14, R19: value 1K -> 4.7K
- X6: device con-ptr500:AK500/2 -> con-ptr500:AK500/6
- X7: device con-ptr500:AK500/2 -> con-ptr500:AK500/3
Connections:
- removed net 13: PCB1.13
- removed net LOW_POWER: PCB1.4
- removed net N$8: JP4.2, PCB1.SDA1
- new net AT_PARK_PIN_EXT: IC5G$1.A7, R20.1, X7-2.KL
- new net AT_PARK_PIN_LOOP_EXT: IC6G$1.B3, R12.1, X7-3.KL
- new net BUF_EN: IC5G$1.*OE, PCB1.A3, R22.2
- new net D13: IC5G$1.B0, PCB1.13
- new net D13_EXT: IC5G$1.A0, R21.2, X8-2.KL
- new net DTR_DSR_DCD: IC3.!DCD, IC3.!DSR, IC3.!DTR
- new net N$1: IC3.!RESET, R11.1, R9.2
- new net N$4: IC5G$1.B4
- new net N$9: XB1.!CTS!/DIO7, XB1.!RTS!/AD6/DIO6
- new net RTS_CTS: IC3.!CTS, IC3.!RTS
- new net RX2: IC3.TXD, PCB1.17(RX2)
- new net SCL: IC1.SCL, PCB1.SCL1, R3.1
- new net SDA: IC1.SDA, PCB1.SDA1, R1.1
- new net TX2: IC3.RXD, PCB1.16(TX2)
- new net USBDM: IC3.USBDM, X13.2
- new net USBDP: IC3.USBDP, X13.3
- new net USB_VCC: R9.1, X13.1
- new net XBEE_DIN: PCB1.18(TX1), XB1.DIN/!CONFIG
- new net XBEE_DOUT: PCB1.19(RX1), XB1.DOUT
- net +12V: now also X11-2.KL; no longer U$2.P$2
- net 3.3V: now also C5.1, C9.1, IC1.VCC, IC3.VCCIO, IC5G$1.DIR, IC5P.VDD, R1.2, R22.1, R3.2, XB1.VCC; no longer IC2P.VDD
- net AT_PARK_PIN: now also IC5G$1.B7; no longer X7-1.KL
- net AT_PARK_PIN_LOOP: now also IC6G$1.A3; no longer X7-2.KL
- net BUTTON_EAST_OPEN: now also IC5G$1.B3; no longer IC2G$1.1Y2
- net BUTTON_EAST_OPEN_5V: now also IC5G$1.A3; no longer IC2G$1.1A2
- net BUTTON_WEST_CLOSE: now also IC5G$1.B2; no longer IC2G$1.2Y1
- net BUTTON_WEST_CLOSE_5V: now also IC5G$1.A2; no longer IC2G$1.2A1
- net GND: now also C5.2, C6.2, C7.2, C8.2, C9.2, IC1.A0, IC1.A1, IC1.A2, IC1.GND, IC3.GND, IC3.GND@1, IC3.GND@2, IC3.GND@A, IC5G$1.A4, IC5P.GND, IC6G$1.*OE, IC6G$1.A4, IC6G$1.A5, IC6G$1.A6, IC6G$1.A7, IC6P.GND, R11.2, X11-1.KL, X12-1.KL, X12-2.KL, X13.4, X13.S1, X13.S2, X7-1.KL, X8-1.KL, XB1.!DTR!/SLEEP_RQ/DI8, XB1.GND; no longer IC2G$1.*1OE, IC2G$1.*2OE, IC2P.GND, U$2.P$1, U$3.P$1, U$3.P$3, U$3.P$5, X6-2.KL
- net HOME_SHUTTER_CLOSED: now also IC5G$1.B1; no longer IC2G$1.2Y0
- net HOME_SHUTTER_CLOSED_5V: now also IC5G$1.A1; no longer IC2G$1.2A0
- net M_DIR: now also IC6G$1.A1; no longer IC2G$1.1A3
- net M_DIR_5V: now also IC6G$1.B1, X6-3.KL; no longer IC2G$1.1Y3, U$3.P$4
- net M_EN: now also IC6G$1.A0; no longer IC2G$1.2A2
- net M_EN_5V: now also IC6G$1.B0, X6-1.KL; no longer IC2G$1.2Y2, U$3.P$2
- net M_STEP: now also IC6G$1.A2; no longer IC2G$1.2A3
- net M_STEP_5V: now also IC6G$1.B2, X6-5.KL; no longer IC2G$1.2Y3, U$3.P$6
- net N$6: now also C8.1, IC3.3V3OUT; no longer JP4.1, PCB1.SCL1
- net RG-11: now also IC5G$1.B5; no longer IC2G$1.1Y1
- net RG-11-IN_5V: now also IC5G$1.A5; no longer IC2G$1.1A1
- net SHUTTER_OPENED: now also IC5G$1.B6; no longer IC2G$1.1Y0
- net SHUTTER_OPENED_5V: now also IC5G$1.A6; no longer IC2G$1.1A0
- net VCC: now also C6.1, C7.1, IC3.VCC, IC6G$1.DIR, IC6P.VDD, R12.2, R20.2, R21.1, X6-2.KL, X6-4.KL, X6-6.KL; no longer X6-1.KL
- net XBEE_RESET: now also XB1.!RESET
Other:
- note added: "3.3V -> 5V"
- note added: "5V->3.3V"
- moved on the sheet: C1, C2, C3, C4, R10, R13, R14, R15, R16, R17, R18, R19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

Commit message: Re-base the code with the dome code
Parts:
- removed PCB1: ARDUINO_DUE_SHIELD_SHORT, arduino_shield:ARDUINO_DUE_SHIELD_SHORT
- removed R22, R9: 4.7K, rti:R-EU'0805'
- removed X12: (no value), con-ptr500:AK500/2
- removed X6: (no value), con-ptr500:AK500/6
- added 25MHZ: CB3LV-OSCILATOR, rti:CB3LV-OSCILATOR
- added C10: 22nF, rcl:C-EUC0805
- added C11, C12, C14, C16, C17, C20: 100nF, rcl:C-EUC0805
- added C13, C18, C22: 10nF, rcl:C-EUC0805
- added C15, C21: 6.8nF, rcl:C-EUC0805
- added C19: 4.7uF, rcl:C-EUC0805
- added C25, C26: 10uF, rcl:C-EUC0805
- added FL1: BLM21AG121SN1D, BLM21AG121SN1D:BLM21AG121SN1D
- added IC4: REG1117, burr-brown:REG1117
- added J2: XT60PW-M, samacsys:XT60PW-M
- added R23: 10 1%, rcl:R-EU_R0805
- added R24, R25, R26, R27: 49.9 1%, rcl:R-EU_R0805
- added R28, R29: 330, rcl:R-EU_R0805
- added R30, R31, R32, R33, R34, R35, R36, R37, R38, R40: 4.7K, rcl:R-EU_R0805
- added R39: 12.4K 1%, rcl:R-EU_R0805
- added U$1: ARDUINO_DUE_SHIELD_FULL, arduino_shield:ARDUINO_DUE_SHIELD_FULL
- added U$2: MCP120T-270I_TT, MCP120T-270I_TT:MCP120T-270I_TT
- added U1: W5500, W5500:W5500
- added X10: (no value), rti:AK500/3
- added X9: J1011F21PNL, rti:J1011F21PNL
- C1, C3: device rti:C-EU'0805' -> rcl:C-EUC0805; MPN (none) -> CC0805KKX5R8BB106
- C2: device rti:CPOL-EU -> rcl:CPOL-EUUD-10X10; MPN (none) -> MAL215099804E3
- C4, C5, C6, C7, C8, C9: device rti:C-EU'0805' -> rcl:C-EUC0805; MPN (none) -> 0805YD104KAT2A
- IC1: device microchip:24AA128ST -> rti:24AA128ST
- IC3: MPN (none) -> FT232RL-REEL
- IC5: MPN (none) -> 74LVC245APW,112
- IC6: device rti:74LVC245 -> rti:74ABT245; MPN (none) -> 74ABT245PW,112
- R1, R3: device rti:R-EU'0805' -> rcl:R-EU_R0805; MPN (none) -> RT0805FRE071KL
- R10, R2, R6, R7, R8: device rti:R-EU'0805' -> rcl:R-EU_R0805; MPN (none) -> AT0805BRD07100KL
- R11: device rti:R-EU'0805' -> rcl:R-EU_R0805; MPN (none) -> RT0805FRE0710KL
- R12, R13, R14, R15, R16, R17, R18, R19, R20, R21, R4: device rti:R-EU'0805' -> rcl:R-EU_R0805; MPN (none) -> RT0805FRE074K7L
- R5: device rti:R-EU'0805' -> rcl:R-EU_R0805; MPN (none) -> RT0805FRD07100RL
- X1, X11, X3, X8: device con-ptr500:AK500/2 -> rti:AK500/2; MPN (none) -> 691101710002
- X13: device con-berg:PN61729-S -> rti:PN61729-S; MPN (none) -> SS-52300-001
- X2: device con-ptr500:AK500/2 -> rti:AK500/3
- X4, X5, X7: device con-ptr500:AK500/3 -> rti:AK500/3; MPN (none) -> 691101710003
- XB1: device maxstream:XBEE -> rti:XBEE
Connections:
- removed net BUF_EN: IC5G$1.*OE, PCB1.A3, R22.2
- removed net N$1: IC3.!RESET, R11.1, R9.2
- new net +3V3: 25MHZ.OE, 25MHZ.VDD, C13.1, C16.1, C20.1, C26.1, C9.1, FL1.2, IC3.VCCIO, IC4.VOUT, R28.2, R29.2, R30.2, R36.2, R37.2, R38.2, U1.VDD
- new net ACT_LED: U1.ACTLED, X9.C-L
- new net AVDD: C11.1, C12.1, C14.1, C17.1, FL1.1, R23.2, R24.2, R25.2, U1.AVDD@1, U1.AVDD@2, U1.AVDD@3, U1.AVDD@4, U1.AVDD@5, U1.AVDD@6
- new net ETH_CS: U$1.52, U1.SCS_N
- new net ETH_RESET: R30.1, U$1.53, U1.RST_N
- new net FTDI_RESET: IC3.!RESET, R11.1, U$1.23
- new net INT_N: U$1.32, U1.INT_N
- new net LINK_ACK: U1.LINKLED, X9.C-R
- new net N$10: R28.1, X9.AL
- new net N$11: C15.2, X9.RD+
- new net N$12: C21.2, X9.RD-
- new net N$13: C10.1, R23.1, X9.CT
- new net N$17: U1.DUPLED
- new net N$22: R31.1, U1.RSVD@2
- new net N$23: R32.1, U1.RSVD@3
- new net N$24: R33.1, U1.RSVD@4
- new net N$25: R34.1, U1.RSVD@5
- new net N$26: R35.1, U1.RSVD@6
- new net N$27: R36.1, U1.PMODE2
- new net N$28: R37.1, U1.PMODE1
- new net N$29: R38.1, U1.PMODE0
- new net N$31: C19.2, U1.TOCAP
- new net N$32: U1.VBG
- new net N$33: C18.2, U1.1V2O
- new net N$34: R39.1, U1.EXRES1
- new net N$35: R40.2, U1.RSVD@1
- new net N$7: C22.1, R26.2, R27.2, X9.CR
- new net N$8: R29.1, X9.A-R
- new net RESET: U$1.RESET, U$2.~RST
- new net RXN: C21.1, R26.1, U1.RXN
- new net RXP: C15.1, R27.1, U1.RXP
- new net SCLK: U$1.SCK, U1.SCLK
- new net SDI: U$1.SDI, U1.MISO
- new net SDO: U$1.SDO, U1.MOSI
- new net TXN: R25.1, U1.TXN, X9.TD-
- new net TXP: R24.1, U1.TXP, X9.TD+
- new net XI: 25MHZ.FO, U1.XI/CLKIN
- new net XO: U1.XO
- net +12V: now also C25.1, IC4.VIN, J2.2, U$1.VIN; no longer PCB1.VIN, X2-1.KL
- net 3.3V: now also U$1.3.3V, U$2.VDD; no longer C9.1, IC3.VCCIO, PCB1.3.3V, R22.1
- net AT_PARK_PIN: now also U$1.A5; no longer PCB1.A5
- net AT_PARK_PIN_LOOP: now also U$1.A4; no longer PCB1.A4
- net BUTTON_EAST_OPEN: now also U$1.5; no longer PCB1.5
- net BUTTON_WEST_CLOSE: now also U$1.6; no longer PCB1.6
- net D13: now also U$1.13; no longer PCB1.13
- net GND: now also 25MHZ.GND, C10.2, C11.2, C12.2, C13.2, C14.2, C16.2, C17.2, C18.1, C19.1, C20.2, C22.2, C25.2, C26.2, IC4.GND, IC5G$1.*OE, J2.1, R31.2, R32.2, R33.2, R34.2, R35.2, R39.2, R40.1, U$1.GND, U$1.GND@2, U$1.GND@3, U$1.GND@4, U$1.GND@5, U$1.GND@6, U$2.VSS, U1.AGND@1, U1.AGND@2, U1.AGND@3, U1.AGND@4, U1.AGND@5, U1.AGND@6, U1.GND, X9.4/NC, X9.5/NC, X9.CGND, X9.CGND2; no longer PCB1.GND, PCB1.GND., PCB1.GND.., X12-1.KL, X12-2.KL, X2-2.KL
- net HOME_SHUTTER_CLOSED: now also U$1.2; no longer PCB1.2
- net M_DIR: now also U$1.11; no longer PCB1.11
- net M_DIR_5V: now also X2-3.KL; no longer X6-3.KL
- net M_EN: now also U$1.10; no longer PCB1.10
- net M_EN_5V: now also X2-1.KL; no longer X6-1.KL
- net M_STEP: now also U$1.12; no longer PCB1.12
- net M_STEP_5V: now also X10-2.KL; no longer X6-5.KL
- net RG-11: now also U$1.7; no longer PCB1.7
- net RX2: now also U$1.17(RX2); no longer PCB1.17(RX2)
- net SCL: now also U$1.SCL1; no longer PCB1.SCL1
- net SDA: now also U$1.SDA1; no longer PCB1.SDA1
- net SHUTTER_OPENED: now also U$1.3; no longer PCB1.3
- net TX2: now also U$1.16(TX2); no longer PCB1.16(TX2)
- net USB_VCC: no longer R9.1
- net VCC: now also U$1.+5V@1, U$1.+5V@3, U$1.+5V@4, X10-1.KL, X10-3.KL, X2-2.KL; no longer PCB1.5V, X6-2.KL, X6-4.KL, X6-6.KL
- net VPIN: now also U$1.A0; no longer PCB1.A0
- net XBEE_DIN: now also U$1.18(TX1); no longer PCB1.18(TX1)
- net XBEE_DOUT: now also U$1.19(RX1); no longer PCB1.19(RX1)
- net XBEE_RESET: now also U$1.8; no longer PCB1.8
